File: EMG-KiCad/_autosave-EMG-KiCad.kicad_sch (KiCad schematic)
At the start: 30 parts, among them J1 Conn_01x03_Socket, J2 Conn_01x03_Socket, U1 AD623, U2 OPA1662D, U3 OPA1662D, U4 OPA1662D, U5 OPA1662D, U6 OPA1662D, U7 LDO 3.3, U8 LDO 1.5

Commit message: Full circuit
Parts:
- added C11, C12, C13, C14, C15, C16, C17, C18: C_Small, symbol Device:C_Small
- added R9: R_Small, symbol Device:R_Small
- added unit 1 of U5
- added U9: OPA1662D, Package_SO:SOIC-8_3.9x4.9mm_P1.27mm, symbol Amplifier_Operational:OPA1662D
Connections:
- net Earth: now also J2.3 (Pin_3), C11.2, C12.2, C13.2, C14.2, C15.2, C16.1, C17.2, C18.2
- net V+: now also C10.1, C9.1, U7.5 (OUT), U8.1 (IN), C12.1, C13.1, C16.2, U9.8 (V+)
- net V-: now also U9.4 (V-)
- net Vref: now also C17.1, C18.1, R9.1, R9.2, U5.1, U5.2 (-)
- net Vout: now reaches C4.2, J2.1 (Pin_1), R10.2, U3.7
- net Vpower: now reaches C8.1, J2.2 (Pin_2), U7.1 (IN)
- net Vpower: now also C11.1
- net at U8.5 (OUT): now also C14.1, C15.1, U5.3 (+)
Other:
- moved on the sheet: C10, C8, C9
